File: pcb/pi_hat.kicad_pcb (KiCad board)
At the start: 2 copper layers, 61.6 x 65.4 mm, 14 parts, among them J10_12Vin1 Screw_Terminal_01x02, J1_ButtonPad1 Conn_01x08, J2 Raspberry pi, J3_5Vin1 Screw_Terminal_01x02, J4_GPIO1 Conn_01x04, J5_I2C1 Conn_01x04, J6_Fan1 Conn_01x04, J7_I2C1 Conn_01x04, J8_RGB_Gnd1 Screw_Terminal_01x04, J9_W_Gnd1 Screw_Terminal_01x02, Q1 IRF540N, Q2 IRF540N, Q3 IRF540N, Q4 IRF540N

Commit message: v2
Parts:
- moved Q3 8.52 mm to (121.3, 88.9), turned to 90 degrees
- moved Q4 8.52 mm to (121.3, 78.1), turned to 90 degrees
- moved Q1 8.52 mm to (121.3, 110.5), turned to 90 degrees
- moved Q2 8.52 mm to (121.3, 99.7), turned to 90 degrees
- moved J6_Fan1 7.24 mm to (104.8, 64.8), turned to 270 degrees
- moved J9_W_Gnd1 5.72 mm to (102.2, 71.1)
- moved J10_12Vin1 1.27 mm to (111.1, 57.1)
- moved J3_5Vin1 1.27 mm to (123.8, 57.1)
Connections:
- J10_12Vin1 pad 1: +12V -> GND
- J10_12Vin1 pad 2: GND -> +12V
- J2 pad 31: /White -> /Blue
- J2 pad 33: /Red -> /Green
- J2 pad 35: /Green -> /Red
- J2 pad 37: /Blue -> /White
- J2 pad 6: Net-(J2-Pad6) -> GND
Routing:
- net /White: track 47.6 -> 106.1 mm
- net /Red: track 37.9 -> 94.4 mm
- net /Green: track 31.1 -> 86.4 mm
- net +12V: track 57.9 -> 38.6 mm
- net Net-(J2-Pad12): track 66.8 -> 80.6 mm
- net Net-(J8_RGB_Gnd1-Pad2): track 11.4 -> 19.6 mm
- net Net-(J8_RGB_Gnd1-Pad3): track 13.8 -> 20.9 mm
- net Net-(J8_RGB_Gnd1-Pad4): track 17.6 -> 23.3 mm
- net Net-(J9_W_Gnd1-Pad2): track 14.1 -> 19.3 mm
- net /Blue: track 28.3 -> 25.4 mm
- net +5V: track 23.8 -> 23.3 mm
- net GND: vias 9 -> 3
Other:
- outline, holes or cut-outs redrawn
