File: pcb/pi_hat.sch (KiCad schematic (older format))
At the start: 14 parts, among them J10_12Vin1 Screw_Terminal_01x02, J1_ButtonPad1 Conn_01x08, J2 Raspberry pi, J3_5Vin1 Screw_Terminal_01x02, J4_GPIO1 Conn_01x04, J5_I2C1 Conn_01x04, J6_Fan1 Conn_01x04, J7_I2C1 Conn_01x04, J8_RGB_Gnd1 Screw_Terminal_01x04, J9_W_Gnd1 Screw_Terminal_01x02, Q1 IRF540N, Q2 IRF540N, Q3 IRF540N, Q4 IRF540N

Commit message: v2
Connections:
- net +12V: now also J10_12Vin1.2 (Pin_2); no longer J10_12Vin1.1 (Pin_1)
- net Blue: now also J2.31 (Pin_31); no longer J2.37 (Pin_37)
- net GND: now also J10_12Vin1.1 (Pin_1), J2.6 (Pin_6); no longer J10_12Vin1.2 (Pin_2)
- net Green: now also J2.33 (Pin_33); no longer J2.35 (Pin_35)
- net Red: now also J2.35 (Pin_35); no longer J2.33 (Pin_33)
- net White: now also J2.37 (Pin_37); no longer J2.31 (Pin_31)
Changed lines of the file:
@@
 L power:GND #PWR0120
 U 1 1 5FCD08CA
+P 9600 1750
+F 0 "#PWR0120" H 9600 1500 50  0001 C CNN
+F 1 "GND" V 9605 1622 50  0000 R CNN
+F 2 "" H 9600 1750 50  0001 C CNN
+F 3 "" H 9600 1750 50  0001 C CNN
+	1    9600 1750
+	0    -1   -1   0
+$EndComp
+$Comp
+L power:+12V #PWR0121
+U 1 1 5FCD14D8
 P 9600 1650
-F 0 "#PWR0120" H 9600 1400 50  0001 C CNN
-F 1 "GND" V 9605 1522 50  0000 R CNN
+F 0 "#PWR0121" H 9600 1500 50  0001 C CNN
+F 1 "+12V" V 9615 1778 50  0000 L CNN
 F 2 "" H 9600 1650 50  0001 C CNN
 F 3 "" H 9600 1650 50  0001 C CNN
 	1    9600 1650
-	0    -1   -1   0
-$EndComp
-$Comp
-L power:+12V #PWR0121
-U 1 1 5FCD14D8
-P 9600 1750
-F 0 "#PWR0121" H 9600 1600 50  0001 C CNN
-F 1 "+12V" V 9615 1878 50  0000 L CNN
-F 2 "" H 9600 1750 50  0001 C CNN
-F 3 "" H 9600 1750 50  0001 C CNN
-	1    9600 1750
 	0    1    1    0
 $EndComp
@@
 Text Label 7500 2300 2    50   ~ 0
 Blue
+Text Label 3150 5800 0    50   ~ 0
+White
+Wire Wire Line
+	3500 5100 3150 5100
+Text Label 3150 5600 0    50   ~ 0
+Red
+Text Label 3150 5400 0    50   ~ 0
+Green
 Text Label 3150 5200 0    50   ~ 0
-White
-Wire Wire Line
-	3500 5100 3150 5100
-Text Label 3150 5400 0    50   ~ 0
-Red
-Text Label 3150 5600 0    50   ~ 0
-Green
-Text Label 3150 5800 0    50   ~ 0
 Blue
 Wire Wire Line
@@
 Wire Wire Line
 	1550 5000 1550 4000
+$Comp
+L power:GND #PWR?
+U 1 1 5FFB8484
+P 3150 2700
+F 0 "#PWR?" H 3150 2450 50  0001 C CNN
+F 1 "GND" V 3155 2572 50  0000 R CNN
+F 2 "" H 3150 2700 50  0001 C CNN
+F 3 "" H 3150 2700 50  0001 C CNN
+	1    3150 2700
+	0    -1   -1   0
+$EndComp
 $EndSCHEMATC
